File: OdytsseySwitch.kicad_pcb (KiCad board)
At the start: 2 copper layers, 112 x 102 mm, 42 parts, among them J1 USB-C, J2 SSD1306_PANEL, J4 QWIIC_I2C, J5 RGB_OUT, J6 EXPANSION, J7 JOYSTICK, SW1 MX_HOTSWAP, SW2 MX_HOTSWAP, SW3 MX_HOTSWAP, SW4 MX_HOTSWAP, SW5 MX_HOTSWAP, SW6 BOOT, SW7 RESET, U1 ESP32-S3-WROOM-1, U3 AP2112K-3.3, U4 USBLC6-2SC6

Commit message: Route the board and clear DRC
Swaps the module connectors from through-hole pin headers to SMD sockets, which
removes the last through-hole parts and drops the assembly's soldering step
entirely. It also fixes a real defect: the board previously carried male pin
headers facing modules that are themselves male, so nothing would have plugged
in.

Routing is autorouted with every net connected, then repaired by hand where the
router left gaps. Ground pours bond solid to pads instead of through thermal
spokes, since starved spokes were stranding pads on a reflow-assembled board,
and 160 stitching vias tie the two pours together. C8 had to move: the router
sealed it into a pocket its ground pad could not escape.

ERC, DRC and schematic parity are all clean, and Gerbers, drill files,
pick-and-place data and the BOM are regenerated to match.

Co-Authored-By: Claude Opus 5 (1M context) <noreply@anthropic.com>
Parts:
- removed C10, C11, C14: 1uF, Capacitor_SMD:C_0603_1608Metric
- removed C12: 2.2uF, Capacitor_SMD:C_0603_1608Metric
- removed C13: 4.7uF, Capacitor_SMD:C_0603_1608Metric
- removed C15: 100nF, Capacitor_SMD:C_0603_1608Metric
- removed R10: 910k, Resistor_SMD:R_0603_1608Metric
- J2: value SSD1306_PANEL -> OLED_I2C; footprint Connector_FFC-FPC:Hirose_FH12-30S-0.5SH_1x30-1MP_P0.50mm_Horizontal -> Connector_PinSocket_2.54mm:PinSocket_1x04_P2.54mm_Vertical_SMD_Pin1Left
- J5: footprint Connector_PinHeader_2.54mm:PinHeader_1x03_P2.54mm_Vertical -> Connector_PinSocket_2.54mm:PinSocket_1x03_P2.54mm_Vertical_SMD_Pin1Left
- J6: footprint Connector_PinHeader_2.54mm:PinHeader_1x08_P2.54mm_Vertical -> Connector_PinSocket_2.54mm:PinSocket_1x08_P2.54mm_Vertical_SMD_Pin1Left
- J7: footprint Connector_PinHeader_2.54mm:PinHeader_1x05_P2.54mm_Vertical -> Connector_PinSocket_2.54mm:PinSocket_1x05_P2.54mm_Vertical_SMD_Pin1Left
- moved C8 3.81 mm to (168.0, 96.5), turned to 0 degrees
Connections:
- J2 pad 2: /OLED_C2N -> +3V3
- J2 pad 3: /OLED_C2P -> /OLED_SCL
- J2 pad 4: /OLED_C1P -> /OLED_SDA
- U1 pad 11: /OLED_RES -> unconnected-(U1-IO18-Pad11)
Routing:
- net +3V3: track 0.00 -> 307.8 mm, vias 0 -> 3
- net VBUS: track 0.00 -> 162.6 mm
- net /OLED_SDA: track 0.00 -> 134.1 mm, vias 0 -> 2
- net /OLED_SCL: track 0.00 -> 121.7 mm, vias 0 -> 2
- net /JOY_VRY: track 0.00 -> 85.2 mm, vias 0 -> 2
- net /JOY_VRX: track 0.00 -> 83.4 mm, vias 0 -> 3
- net /RGB_DIN_MCU: track 0.00 -> 74.9 mm, vias 0 -> 2
- net /EN: track 0.00 -> 72.8 mm
- net /JOY_SW: track 0.00 -> 72.0 mm, vias 0 -> 2
- net /BOOT_N: track 0.00 -> 70.9 mm
- net /EXP_GPIO10: track 0.00 -> 64.2 mm, vias 0 -> 2
- net /UART_TX: track 0.00 -> 63.1 mm, vias 0 -> 2
- net /USB_DM_MCU: track 0.00 -> 56.3 mm
- net /UART_RX: track 0.00 -> 54.7 mm, vias 0 -> 2
- net /USB_DP_MCU: track 0.00 -> 51.8 mm, vias 0 -> 2
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
Commit message: Pull a stitching via clear of the USB-C shield hole
Measuring the design against typical fab capability turned up one hole pair at
0.286 mm, well under the 0.5 mm most houses ask for: a ground stitching via had
landed beside J1's shield post. Removing it costs nothing, since the pours stay
tied through the remaining two hundred vias and connectivity is unchanged.

Tightest hole spacing is now 0.440 mm, and every pair at that figure is inside
a Kailh hotswap footprint, where the peg and stem holes are milled rather than
drilled.

Fabrication outputs regenerated.

Co-Authored-By: Claude Opus 5 (1M context) <noreply@anthropic.com>
Routing:
- net GND: vias 163 -> 162
Changed lines of the file:
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@@
 		)
 		(fp_text user "${REFERENCE}"
-			(at 0 0 360)
+			(at 0 0 0)
 			(layer "B.Fab")
 			(effects
@@
 		(size 0.6)
 		(drill 0.3)
-		(layers "F.Cu" "B.Cu")
-		(net "GND")
-	)
-	(via
-		(at 133.531919 62.61675)
-		(size 0.6)
-		(drill 0.3)
